File: Main/PCB/Display badge.kicad_pcb (KiCad board)
At the start: 2 copper layers, 70.3 x 70.2 mm, 69 parts, among them J1 TYPE-C-31-M-12, J2 FFC2B28-12-G, J3 Conn_01x03, J4 DM3AT-SF-PEJM5, M1 C0720B001F, Q1 2N7002, SW1 PTS810_SJM_250_SMTR_LFS, SW2 PTS810_SJM_250_SMTR_LFS, SW3 PTS810_SJM_250_SMTR_LFS, SW4 PTS810_SJM_250_SMTR_LFS, SW5 PTS810_SJM_250_SMTR_LFS, U1 AMS1117-3.3, U2 ESP32-S3-WROOM-1-N16R2, U3 BMI270, U4 DRV2605LDGST

Commit message: ZINE IS OUT
Parts:
- added REF**: screen, Vibrator:screen, F.Cu at (85.4, 104.8)
- added REF**: screen, Vibrator:screen, F.Cu at (86.3, 106.4)
- moved REF** 1.00 mm to (65.6, 117.8)
- moved REF** 1.00 mm to (60.6, 81.4)
- moved REF** 1.00 mm to (97.2, 127.4)
- moved REF** 1.00 mm to (109.8, 80.8)
